File: LHRE_Button_PCB_V1.kicad_pcb (KiCad board)
At the start: 2 copper layers, 124.1 x 58.3 mm, 70 parts, among them IC1 LM5155DSSR, IC2 LM5155DSSR, J1 Conn_01x12_Female, J2 Conn_01x12_Female, J3 Conn_01x02_Female, J4 Conn_01x02_Female, Q1 CSD18537NQ5A, Q2 CSD18537NQ5A, SW1 Dashboard_Button, SW2 Dashboard_Button, SW3 Dashboard_Button, SW4 Dashboard_Button, SW5 Dashboard_Button, SW6 Dashboard_Button

Commit message: updated dash PCB
Parts:
- removed the J3 at (112.8, 44.5)
- added H1: MountingHole, MountingHole:MountingHole_3.5mm, F.Cu at (83.8, 39.8)
- added H2: MountingHole, MountingHole:MountingHole_3.5mm, F.Cu at (83.8, 78.4)
- added H3: MountingHole, MountingHole:MountingHole_3.5mm, F.Cu at (152.4, 39.8)
- added H4: MountingHole, MountingHole:MountingHole_3.5mm, F.Cu at (152.4, 110.9)
- added H5: MountingHole, MountingHole:MountingHole_3.5mm, F.Cu at (168.8, 39.8)
- added H6: MountingHole, MountingHole:MountingHole_3.5mm, F.Cu at (222.7, 39.8)
- added H7: MountingHole, MountingHole:MountingHole_3.5mm, F.Cu at (168.8, 110.9)
- added H8: MountingHole, MountingHole:MountingHole_3.5mm, F.Cu at (222.7, 78.4)
- added J4: Conn_01x02_Female, Connector_Wire:SolderWire-0.75sqmm_1x02_P4.8mm_D1.25mm_OD2.3mm, F.Cu at (179.1, 47.0)
- D1, D2: footprint Dashboard_LED:LEDC1608X80N -> Connector_Wire:SolderWire-0.75sqmm_1x02_P4.8mm_D1.25mm_OD2.3mm
- moved J1 113.3 mm to (149.5, 67.2), turned to -90 degrees
- moved D2 101.5 mm to (221.0, 61.4), turned to 90 degrees
- moved R8 92.9 mm to (210.2, 52.7)
- moved SW4 77.5 mm to (199.9, 44.8)
- moved R6 77.4 mm to (204.7, 60.5)
- moved SW5 77.4 mm to (199.9, 65.1)
- moved SW6 77.3 mm to (199.9, 85.4)
- moved R7 77.2 mm to (204.6, 80.7)
- moved R5 77.1 mm to (204.4, 40.2)
- moved R13 72.3 mm to (140.7, 99.8)
- moved C10 72.3 mm to (137.3, 99.9)
- moved C3 72.3 mm to (142.3, 104.4)
- moved C5 72.3 mm to (135.3, 99.9)
- moved R10 72.3 mm to (138.9, 104.4)
- moved R14 72.3 mm to (142.5, 99.8)
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- renumbered J4 to J3
Connections:
- J1 pad 1: GND1 -> AMS
- J1 pad 10: MCU_SIG1 -> SW3_OUT
- J1 pad 11: 12V_L -> Vin_L
- J1 pad 12: AMS -> GND1
- J1 pad 2: Vin_L -> 12V_L
- J1 pad 3: SW3_OUT -> MCU_SIG1
- J1 pad 4: MCU_SIG3 -> SW1_OUT
- J1 pad 6: SW2_OUT -> MCU_SIG2
- J1 pad 7: MCU_SIG2 -> SW2_OUT
- J1 pad 9: SW1_OUT -> MCU_SIG3
Routing:
- net 12V_L: track 100.6 -> 181.4 mm
- net MCU_SIG3: track 13.7 -> 60.9 mm, vias 0 -> 2
- net AMS: track 15.7 -> 58.3 mm
- net SW2_OUT: track 21.8 -> 60.6 mm
- net MCU_SIG2: track 10.1 -> 46.6 mm
- net SW1_OUT: track 25.6 -> 59.4 mm
- net MCU_SIG1: track 13.2 -> 46.6 mm
- net 12V_R: track 107.8 -> 139.7 mm, vias 0 -> 2
- net MCU_SIG6: track 12.9 -> 41.8 mm
- net GND: track 84.7 -> 55.8 mm
- net SW6_OUT: track 24.9 -> 50.9 mm
- net SW4_OUT: track 29.7 -> 51.8 mm
- net Net-(IC2-Pad3): track 12.7 -> 34.2 mm, vias 2 -> 0
- net Net-(Q2-Pad1): track 9.92 -> 31.4 mm
- net MCU_SIG4: track 17.1 -> 37.7 mm
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Other:
- board size 124.1 x 58.3 mm -> 146.5 x 78.7 mm
